Commit message: fix: complete phase two ros gz integration

File: src/sentry_gazebo_2024/m_bot/mbot_description/sensors/hdl32e.xacro (robot description, xacro)
@@ -4,7 +4,7 @@
   <xacro:macro name="hdl32e" params="parent *origin">
     <joint name="velodyne_base_joint" type="fixed"><xacro:insert_block name="origin"/><parent link="${parent}"/><child link="velodyne_base"/></joint>
-    <link name="velodyne_base"><visual><geometry><mesh filename="package://mbot_description/meshes/HDL32E_base.dae"/></geometry></visual></link>
+    <link name="velodyne_base"><visual><geometry><mesh filename="file://$(find mbot_description)/meshes/HDL32E_base.dae"/></geometry></visual></link>
     <joint name="velodyne_joint" type="fixed"><origin xyz="0 0 0.09081"/><parent link="velodyne_base"/><child link="velodyne"/></joint>
-    <link name="velodyne"><visual><origin xyz="0 0 -0.09081"/><geometry><mesh filename="package://mbot_description/meshes/HDL32E_scan.dae"/></geometry></visual></link>
+    <link name="velodyne"><visual><origin xyz="0 0 -0.09081"/><geometry><mesh filename="file://$(find mbot_description)/meshes/HDL32E_scan.dae"/></geometry></visual></link>
     <gazebo reference="${parent}">
       <sensor name="velodyne-HDL32E" type="gpu_lidar">

File: src/sentry_gazebo_2024/m_bot/mbot_description/urdf/xacro/gazebo/mbot_base_gazebo.xacro (robot description, xacro)
@@ -104,5 +104,5 @@
         </gazebo>
     </xacro:macro>
-    <xacro:macro name="mbot_base_gazebo" params="color_car">
+    <xacro:macro name="mbot_base_gazebo" params="color_car use_ros2_control:=false">
         <link name="base_footprint">
             <visual>
@@ -144,26 +144,36 @@
         <xacro:caster prefix="front" reflect="-1"/>
         <xacro:caster prefix="back"  reflect="1"/>
-        <!-- controller -->
-        <gazebo>
-            <plugin name="differential_drive_controller"
-                    filename="gz-sim-diff-drive-system">
-                <left_joint>left_wheel_joint</left_joint>
-                <right_joint>right_wheel_joint</right_joint>
-                <wheel_separation>${wheel_joint_y*2}</wheel_separation>
-                <wheel_radius>${wheel_radius}</wheel_radius>
-                <topic>cmd_vel</topic>
-                <odom_topic>odom</odom_topic>
-                <tf_topic>tf</tf_topic>
-                <frame_id>odom</frame_id>
-                <child_frame_id>base_footprint</child_frame_id>
-                <odom_publish_frequency>100.0</odom_publish_frequency>
-            </plugin>
-        </gazebo>
-        <!-- ROS2 control path; controller names and velocity interfaces match legacy. -->
-        <ros2_control name="MbotSystem" type="system">
-            <hardware><plugin>gz_ros2_control/GazeboSimSystem</plugin></hardware>
-            <joint name="left_wheel_joint"><command_interface name="velocity"/><state_interface name="position"/><state_interface name="velocity"/></joint>
-            <joint name="right_wheel_joint"><command_interface name="velocity"/><state_interface name="position"/><state_interface name="velocity"/></joint>
-        </ros2_control>
+        <!-- DiffDrive and gz_ros2_control must not claim the same wheel joints. -->
+        <xacro:unless value="${use_ros2_control}">
+            <gazebo>
+                <plugin name="gz::sim::systems::DiffDrive"
+                        filename="gz-sim-diff-drive-system">
+                    <left_joint>left_wheel_joint</left_joint>
+                    <right_joint>right_wheel_joint</right_joint>
+                    <wheel_separation>${wheel_joint_y*2}</wheel_separation>
+                    <wheel_radius>${wheel_radius}</wheel_radius>
+                    <topic>cmd_vel</topic>
+                    <odom_topic>odom</odom_topic>
+                    <tf_topic>tf</tf_topic>
+                    <frame_id>odom</frame_id>
+                    <child_frame_id>base_footprint</child_frame_id>
+                    <odom_publish_frequency>100.0</odom_publish_frequency>
+                </plugin>
+            </gazebo>
+        </xacro:unless>
+        <xacro:if value="${use_ros2_control}">
+            <!-- Optional control backend; DiffDrive remains the default backend. -->
+            <ros2_control name="MbotSystem" type="system">
+                <hardware><plugin>gz_ros2_control/GazeboSimSystem</plugin></hardware>
+                <joint name="left_wheel_joint"><command_interface name="velocity"/><state_interface name="position"/><state_interface name="velocity"/></joint>
+                <joint name="right_wheel_joint"><command_interface name="velocity"/><state_interface name="position"/><state_interface name="velocity"/></joint>
+            </ros2_control>
+            <gazebo>
+                <plugin name="gz_ros2_control::GazeboSimROS2ControlPlugin" filename="gz_ros2_control-system">
+                    <parameters>$(find mbot_control)/config/mbot_control.yaml</parameters>
+                    <ros><namespace>/mbot</namespace></ros>
+                </plugin>
+            </gazebo>
+        </xacro:if>
     </xacro:macro>
 </robot>

File: src/sentry_gazebo_2024/m_bot/mbot_description/urdf/xacro/gazebo/mbot_gazebo.xacro (robot description, xacro)
@@ -2,5 +2,6 @@
 <!-- ROS2 migration of legacy/.../urdf/xacro/gazebo/mbot_gazebo.xacro. -->
 <robot name="mbot" xmlns:xacro="http://www.ros.org/wiki/xacro">
+    <xacro:arg name="use_ros2_control" default="false"/>
     <xacro:include filename="$(find mbot_description)/urdf/xacro/gazebo/mbot_base_gazebo.xacro" />
-    <xacro:mbot_base_gazebo color_car="Yellow" />
+    <xacro:mbot_base_gazebo color_car="Yellow" use_ros2_control="$(arg use_ros2_control)" />
 </robot>

File: src/sentry_gazebo_2024/m_bot/mbot_description/urdf/xacro/gazebo/mbot_velodyne.xacro (robot description, xacro)
@@ -2,9 +2,10 @@
 <!-- ROS2/Harmonic blue lidar model; legacy geometry and offsets retained. -->
 <robot name="mbot" xmlns:xacro="http://www.ros.org/wiki/xacro">
+    <xacro:arg name="use_ros2_control" default="false"/>
     <xacro:include filename="$(find mbot_description)/urdf/xacro/gazebo/mbot_base_gazebo.xacro" />
     <xacro:property name="lidar_offset_x" value="0" />
     <xacro:property name="lidar_offset_y" value="0" />
     <xacro:property name="lidar_offset_z" value="0.080" />
-    <xacro:mbot_base_gazebo color_car="Blue"/>
+    <xacro:mbot_base_gazebo color_car="Blue" use_ros2_control="$(arg use_ros2_control)"/>
     <!-- lidar VLP-16 -->
     <!-- <xacro:include filename="$(find velodyne_description)/urdf/VLP-16.urdf.xacro" />

File: src/sentry_gazebo_2024/m_bot/mbot_description/urdf/xacro/gazebo/mbot_velodyne_target.xacro (robot description, xacro)
@@ -2,9 +2,10 @@
 <!-- ROS2/Harmonic red target model; legacy geometry and offsets retained. -->
 <robot name="mbot_target" xmlns:xacro="http://www.ros.org/wiki/xacro">
+    <xacro:arg name="use_ros2_control" default="false"/>
     <xacro:include filename="$(find mbot_description)/urdf/xacro/gazebo/mbot_base_gazebo.xacro" />
     <xacro:property name="lidar_offset_x" value="0" />
     <xacro:property name="lidar_offset_y" value="0" />
     <xacro:property name="lidar_offset_z" value="0.080" />
-    <xacro:mbot_base_gazebo color_car="Red"/>
+    <xacro:mbot_base_gazebo color_car="Red" use_ros2_control="$(arg use_ros2_control)"/>
     <!-- lidar VLP-16 -->
     <!-- <xacro:include filename="$(find velodyne_description)/urdf/VLP-16.urdf.xacro" />
